Commit message: completed robot build, understand frame connections, and xacros
the build is interesting, just need to remember what needs to change

File: ros_workspace/src/erl1/urdf/erl1.xacro (robot description, xacro)
@@ -4,4 +4,7 @@
     <xacro:property name="length_wheel" value="0.05" />
     <xacro:property name="radius_wheel" value="0.1" />
+    <xacro:property name="length_prism" value="0.03" />
+    <xacro:property name="width_prism" value="0.03" />
+    <xacro:property name="height_prism" value="0.6" />
     <!-- Macros -->
     <xacro:macro name="default_inertial" params="mass">
@@ -15,4 +18,14 @@
         </inertial>
     </xacro:macro>
+    <xacro:macro name="default_interial_box" params="mass">
+        <inertial>
+            <mass value="${mass}" />
+            <origin rpy="0 0 0" xyz="0 0 0.3"/>
+            <inertia
+                ixx="${mass*(length_prism**2+width_prism**2)/12}" ixy="0" ixz="0"
+                iyy="${mass*(length_prism**2+height_prism**2)/12}" iyz="0"
+                izz="${mass*(length_prism**2+width_prism**2)/12}"/>
+        </inertial>
+    </xacro:macro>
     <xacro:macro name="wheel_geometry">
         <geometry>
@@ -20,4 +33,10 @@
         </geometry>
     </xacro:macro>
+    <xacro:macro name="prism_geometry">
+        <geometry>
+            <box size="${length_prism} ${width_prism} ${height_prism}"/>
+        </geometry>
+    </xacro:macro>
+    <!-- Colors -->
     <material name="blue">
         <color rgba="0.203125 0.23828125 0.28515625 1.0"/>
@@ -109,4 +128,30 @@
                 <box size="0.09 0.09 0.09"/>
             </geometry>
+            <material name="orange"/>
+        </visual>
+    </link>
+    <!-- link 1 -->
+    <link name="link_1">
+        <xacro:default_interial_box mass="2.0"/>
+        <collision>
+            <origin xyz="0 0 0.3" rpy="0 0 0"/>
+            <xacro:prism_geometry/>
+        </collision>
+        <visual name="link_visual">
+            <origin xyz="0 0 0.3" rpy="0 0 0"/>
+            <xacro:prism_geometry/>
+            <material name="orange"/>
+        </visual>
+    </link>
+    <!-- link 2 -->
+    <link name="link_2">
+        <xacro:default_interial_box mass="2.0"/>
+        <collision>
+            <origin xyz="0 0 0.3" rpy="0 0 0"/>
+            <xacro:prism_geometry/>
+        </collision>
+        <visual name="link_visual">
+            <origin xyz="0 0 0.3" rpy="0 0 0"/>
+            <xacro:prism_geometry/>
             <material name="orange"/>
         </visual>
@@ -132,5 +177,5 @@
         <dynamics damping="1.0" friction="1.0"/>
     </joint>
-    <!-- Base -->
+    <!-- Joint Base -->
     <joint type="continuous"
         name="base_joint">
@@ -142,3 +187,23 @@
         <dynamics damping="1.0" friction="1.0"/>
     </joint>
+     <!-- Joint Link 1 -->
+    <joint type="revolute"
+        name="link_1_joint">
+        <origin xyz="0 0 0.045" rpy="0 0 0"/>
+        <child link="link_1"/>
+        <parent link="base"/>
+        <axis xyz="1 0 0"/>
+        <limit lower="-0.785" upper="0.785" effort="100" velocity="10"/>
+        <dynamics damping="1.0" friction="1.0"/>
+    </joint>
+     <!-- Joint Link 2 -->
+    <joint type="revolute"
+        name="link_2_joint">
+        <origin xyz="0.03 0 0.5" rpy="0 0 0"/>
+        <child link="link_2"/>
+        <parent link="link_1"/>
+        <axis xyz="1 0 0"/>
+        <limit lower="-0.785" upper="0.785" effort="100" velocity="10"/>
+        <dynamics damping="1.0" friction="1.0"/>
+    </joint>
 </robot>

Commit message: gazebo-ros bridge

File: ros_workspace/src/erl1/urdf/erl1.xacro (robot description, xacro)
@@ -25,5 +25,5 @@
             <origin rpy="0 0 0" xyz="0 0 0.3"/>
             <inertia
-                ixx="${mass*(length_prism**2+width_prism**2)/12}" ixy="0" ixz="0"
+                ixx="${mass*(width_prism**2+height_prism**2)/12}" ixy="0" ixz="0"
                 iyy="${mass*(length_prism**2+height_prism**2)/12}" iyz="0"
                 izz="${mass*(length_prism**2+width_prism**2)/12}"/>
@@ -90,5 +90,5 @@
         <xacro:default_inertial mass="5.0"/>
         <collision>
-            <origin xyz="0 0 0" rpy="0 0.1570 1.5707"/>
+            <origin xyz="0 0 0" rpy="0 1.5707 1.5707"/>
             <xacro:wheel_geometry/>
         </collision>
@@ -146,5 +146,5 @@
         </visual>
     </link>
-    <!-- link 2 -->
+    <!-- Link 2 -->
     <link name="link_2">
         <xacro:default_interial_box mass="2.0"/>
@@ -158,4 +158,30 @@
             <material name="orange"/>
         </visual>
+    </link>
+    <!-- Camera -->
+    <link name="camera_link">
+        <visual name="camera_link">
+            <origin xyz="0 0 0.05" rpy="0 0 0"/>
+            <geometry>
+                <box size="0.1 0.1 0.1"/>
+            </geometry>
+            <material name="blue"/>
+        </visual>
+        <collision>
+        <origin xyz="0 0 0.05" rpy="0 0 0"/>
+            <geometry>
+                <box size="0.1 0.1 0.1"/>
+            </geometry>
+        </collision>
+        <inertial>
+            <mass value="0.3"/>
+            <origin xyz="0 0 0.05" rpy="0 0 0"/>
+            <inertia
+                ixx="0.0005" ixy="0" ixz="0"
+                iyy="0.0005" iyz="0"
+                izz="0.0005"/>
+            </inertial>
+    </link>
+    <link name="camera_link_optical">
     </link>
     <!-- Joints Right Wheel -->
@@ -209,3 +235,18 @@
         <dynamics damping="1.0" friction="1.0"/>
     </joint>
+    <!-- Joint Camera-->
+    <joint name="camera_joint" type="revolute">
+        <parent link="link_chassis"/>
+        <child link="camera_link"/>
+        <origin xyz="0 0 0.035" rpy="0 0 0"/>
+        <axis xyz="0 0 1"/>
+        <limit lower="-1.57" upper="1.57" effort="5"
+        velocity="1.0"/>
+    </joint>
+    <joint type="fixed"
+        name="camera_optical_joint">
+        <origin xyz="0 0 0" rpy="-1.5707 0 -1.5707"/>
+        <child link="camera_link_optical"/>
+        <parent link="camera_link"/>
+    </joint>
 </robot>

Commit message: IMU, EKF, ODOM

File: ros_workspace/src/erl1/urdf/erl1.xacro (robot description, xacro)
@@ -117,5 +117,5 @@
             <mass value="2.0"/>
             <origin rpy="0 0 0" xyz="0 0 0"/>
-            <inertia ixx="0" ixy="0" ixz="0" iyy="0" iyz="0" izz="0"/>
+            <inertia ixx="0.0027" ixy="0" ixz="0" iyy="0.0027" iyz="0" izz="0.0027"/>
         </inertial>
         <collision>
@@ -184,4 +184,7 @@
     </link>
     <link name="camera_link_optical">
+    </link>
+    <!-- IMU -->
+    <link name="imu_link">
     </link>
     <!-- Joints Right Wheel -->
@@ -236,5 +239,6 @@
     </joint>
     <!-- Joint Camera-->
-    <joint name="camera_joint" type="revolute">
+    <joint type="revolute"
+        name="camera_joint">
         <parent link="link_chassis"/>
         <child link="camera_link"/>
@@ -250,3 +254,9 @@
         <parent link="camera_link"/>
     </joint>
+    <!-- IMU -->
+    <joint name="imu_joint" type="fixed">
+        <origin xyz="0 0 0" rpy="0 0 0" />
+        <parent link="link_chassis"/>
+        <child link="imu_link" />
+    </joint>
 </robot>

Commit message: added GPS + Lidar

File: ros_workspace/src/erl1/urdf/erl1.xacro (robot description, xacro)
@@ -187,4 +187,37 @@
     <!-- IMU -->
     <link name="imu_link">
+        <inertial>
+            <mass value="1e-5"/>
+            <origin xyz="0 0 0" rpy="0 0 0"/>
+            <inertia ixx="1e-6" ixy="0" ixz="0" iyy="1e-6" iyz="0" izz="1e-6"/>
+        </inertial>
+    </link>
+    <!-- GPS -->
+    <link name="navsat_link">
+        <inertial>
+            <mass value="1e-5"/>
+            <origin xyz="0 0 0" rpy="0 0 0"/>
+            <inertia ixx="1e-6" ixy="0" ixz="0" iyy="1e-6" iyz="0" izz="1e-6"/>
+        </inertial>
+    </link>
+    <!-- LiDar -->
+    <link name='scan_link'>
+        <inertial>
+            <mass value="1e-5"/>
+            <origin xyz="0 0 0" rpy="0 0 0"/>
+            <inertia ixx="1e-6" ixy="0" ixz="0" iyy="1e-6" iyz="0" izz="1e-6"/>
+        </inertial>
+        <collision name='collision'>
+            <origin xyz="0 0 0" rpy="0 0 0"/>
+            <geometry>
+                <box size=".1 .1 .1"/>
+            </geometry>
+        </collision>
+        <visual name='scan_link_visual'>
+            <origin xyz="0 0 0" rpy="0 0 0"/>
+            <geometry>
+                <cylinder radius="0.05" length="0.1"/>
+            </geometry>
+        </visual>
     </link>
     <!-- Joints Right Wheel -->
@@ -260,3 +293,15 @@
         <child link="imu_link" />
     </joint>
+    <!-- GPS -->
+    <joint name="navsat_joint" type="fixed">
+        <origin xyz="0 0 0" rpy="0 0 0"/>
+        <parent link="link_chassis"/>
+        <child link="navsat_link" />
+    </joint>
+    <!-- LiDar -->
+    <joint type="fixed" name="scan_joint">
+        <origin xyz="-0.2 0 0.19" rpy="0 0 0"/>
+        <child link="scan_link"/>
+        <parent link="link_chassis"/>
+    </joint>
 </robot>

Commit message: camera sensor, open cv to convert images

File: ros_workspace/src/erl1/urdf/erl1.xacro (robot description, xacro)
@@ -133,30 +133,4 @@
         </visual>
     </link>
-    <!-- link 1 -->
-    <link name="link_1">
-        <xacro:default_interial_box mass="2.0"/>
-        <collision>
-            <origin xyz="0 0 0.3" rpy="0 0 0"/>
-            <xacro:prism_geometry/>
-        </collision>
-        <visual name="link_visual">
-            <origin xyz="0 0 0.3" rpy="0 0 0"/>
-            <xacro:prism_geometry/>
-            <material name="orange"/>
-        </visual>
-    </link>
-    <!-- Link 2 -->
-    <link name="link_2">
-        <xacro:default_interial_box mass="2.0"/>
-        <collision>
-            <origin xyz="0 0 0.3" rpy="0 0 0"/>
-            <xacro:prism_geometry/>
-        </collision>
-        <visual name="link_visual">
-            <origin xyz="0 0 0.3" rpy="0 0 0"/>
-            <xacro:prism_geometry/>
-            <material name="orange"/>
-        </visual>
-    </link>
     <!-- Camera -->
     <link name="camera_link">
@@ -251,24 +225,4 @@
         <dynamics damping="1.0" friction="1.0"/>
     </joint>
-     <!-- Joint Link 1 -->
-    <joint type="revolute"
-        name="link_1_joint">
-        <origin xyz="0 0 0.045" rpy="0 0 0"/>
-        <child link="link_1"/>
-        <parent link="base"/>
-        <axis xyz="1 0 0"/>
-        <limit lower="-0.785" upper="0.785" effort="100" velocity="10"/>
-        <dynamics damping="1.0" friction="1.0"/>
-    </joint>
-     <!-- Joint Link 2 -->
-    <joint type="revolute"
-        name="link_2_joint">
-        <origin xyz="0.03 0 0.5" rpy="0 0 0"/>
-        <child link="link_2"/>
-        <parent link="link_1"/>
-        <axis xyz="1 0 0"/>
-        <limit lower="-0.785" upper="0.785" effort="100" velocity="10"/>
-        <dynamics damping="1.0" friction="1.0"/>
-    </joint>
     <!-- Joint Camera-->
     <joint type="revolute"
